File: h523-obd2-board.kicad_pcb (KiCad board)
At the start: 2 copper layers, 80 x 35 mm, 68 parts, among them J1 Conn_02x05_Odd_Even, J2 Conn_01x03, J3 Conn_01x03, J4 Conn_01x03, J5 Conn_01x03, J6 Conn_01x03, J7 Conn_01x03, J8 Conn_01x03, J9 Conn_01x03, Q1 AO3400A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

Commit message: PROTO A manufactured
Parts:
- removed U5: ADXL345, JLCLibrary:ADXL345
- added C18: 6.8n, Capacitor_SMD:C_0402_1005Metric, F.Cu at (147.3, 79.2)
- added C19: 6.8n, Capacitor_SMD:C_0402_1005Metric, F.Cu at (147.2, 80.3)
- added J10: Conn_01x08, Connector_PinHeader_2.54mm:PinHeader_1x08_P2.54mm_Vertical, F.Cu at (140.7, 52.0)
- added R36: 4.7k, Resistor_SMD:R_0402_1005Metric, F.Cu at (152.9, 80.8)
- added R37: 4.7k, Resistor_SMD:R_0402_1005Metric, F.Cu at (150.9, 80.8)
- C14: value 100nF -> 100n
- C15, C16: value 100n -> 6.8n
- C17: value 1u -> 6.8n; footprint Capacitor_SMD:C_0603_1608Metric -> Capacitor_SMD:C_0402_1005Metric
- moved C15 15.2 mm to (148.8, 67.0), turned to 90 degrees
- moved C17 13.5 mm to (147.2, 78.2), turned to 0 degrees
- moved C16 5.50 mm to (147.3, 77.1), turned to 0 degrees
- moved R29 4.89 mm to (154.4, 79.8), turned to 0 degrees
- moved R28 2.34 mm to (154.4, 78.7), turned to 0 degrees
- moved C12 0.32 mm to (151.8, 76.7)
Connections:
- C15 pad 1: +3V3 -> GND
- C15 pad 2: GND -> ADC1_MCU
- C16 pad 1: +3V3 -> GND
- C16 pad 2: GND -> ADC2_MCU
- C17 pad 1: +3V3 -> GND
- C17 pad 2: GND -> ADC3_MCU
Routing:
- net ADXL_I2C_SCL: track 16.4 -> 76.2 mm, vias 0 -> 1
- net ADXL_I2C_SDA: track 14.3 -> 73.2 mm, vias 2 -> 3
- net GND: track 128.4 -> 120.5 mm, vias 49 -> 48
- net LCD_I2C_SCL: track 51.4 -> 58.1 mm
- net ADC5_MCU: track 41.1 -> 47.5 mm
- net ADC4_MCU: track 36.3 -> 41.9 mm
- net ADC3_MCU: track 33.5 -> 38.5 mm
- net ADC2_MCU: track 31.4 -> 35.7 mm
- net LCD_I2C_SDA: track 55.2 -> 58.2 mm
- net +3V3: track 204.9 -> 207.8 mm, vias 10 -> 12
- net ADC1_MCU: track 14.0 -> 14.8 mm
Other:
- board text added: "3v3 GND"
- board text added: "ADXL345 Module 21x16 circuitrocks/makerlab"
- board text added: "OBD2 Modbus Logger PROTO A"
- board text added: "Pin8 of port on this side"
- board text removed: "-->"
- board text removed: "ADXL G meter"
- board text removed: "OBD2 Modbus Logger PROTO A Luis Alvarez"
- board text removed: "Pin8 of each port on this side"
- board text removed: "X"
- board text removed: "Y"
